Commit message: add ros control for all robotic joints
add gazebo tags

including transmissions

File: robotiq_3f_gripper_visualization/cfg/robotiq-3f-gripper_actuated_gazebo.xacro (robot description, xacro)
@@ -4,20 +4,26 @@
 -->
 <robot name="robotiq-3f-gripper_actuated_gazebo" xmlns:xacro="http://ros.org/wiki/xacro">
-    <xacro:include filename="$(find robotiq_3f_gripper_visualization)/cfg/robotiq_hand_macro.urdf.xacro" />
+    <xacro:include filename="$(find robotiq_3f_gripper_visualization)/cfg/robotiq-3f-gripper_articulated_macro.xacro" />
+    <gazebo>
+        <plugin name="gazebo_ros_control" filename="libgazebo_ros_control.so" />
+    </gazebo>
     <link name="world"/>
-    <xacro:robotiq_hand prefix="" parent="world" reflect="">
-      <origin xyz="0 0 0.5" rpy="0 0 0"/>
-    </xacro:robotiq_hand>
-  <gazebo>
-    <!-- plugin for the RobotiQ hand -->
+    <xacro:robotiq-3f-gripper_articulated prefix="s_model_"/>
+    <joint name="gripper_joint" type="fixed">
+        <parent link="world" />
+        <child link = "s_model_palm" />
+        <origin xyz="0.057 0.0 0.0" rpy="0.0 ${pi} ${-pi/2}" />
+    </joint>
+<!--  <gazebo>
+    <!- - plugin for the RobotiQ hand - ->
     <plugin name="robotiq_hand_plugin" filename="libRobotiqHandPlugin.so">
       <kp_position>10.0</kp_position>
       <kd_position>0.5</kd_position>
-      <!-- Some optional parameters. Check the plugin header file for all of them. -->
-      <!--<prefix>pre_</prefix>-->
-      <!-- This is chosen, so it's compatible with the "Robotiq3FGripperSimpleController.py"-->
+      <!- - Some optional parameters. Check the plugin header file for all of them. - ->
+      <!- -<prefix>pre_</prefix>- ->
+      <!- - This is chosen, so it's compatible with the "Robotiq3FGripperSimpleController.py"- ->
       <topic_command>/Robotiq3FGripperRobotOutput</topic_command>
-      <!-- <topic_state>/hand/state</topic_state> -->
+      <!- - <topic_state>/hand/state</topic_state> - ->
     </plugin>
-  </gazebo>
+  </gazebo> -->
 </robot>

File: robotiq_3f_gripper_visualization/cfg/robotiq-3f-gripper_articulated_macro.xacro (robot description, xacro)
@@ -1,2 +1,3 @@
+<?xml version="1.0"?>
 <!--
 robotiq-3f-gripper_articulated_macro(prefix)
@@ -29,5 +30,14 @@
 				</material>
 			</collision>
+             <inertial>
+            <origin xyz="0 0 0" rpy="0 0 0"/>
+            <mass value="1.3"/>
+            <inertia ixx="0.0035" ixy="0" ixz="-0" iyy="0.0035" iyz="0" izz="0.0035" />
+            </inertial>
 		</link>
+        <gazebo reference="${prefix}palm">
+        <mu1>1.1</mu1>
+        <mu2>1.1</mu2>
+        </gazebo>
 		<link name="${prefix}tool0"/>
         <inertial>
@@ -58,5 +68,5 @@
 			<origin xyz="0.0455 0.0214 0" rpy="0 0 1.57"/>
 		</joint>
-		<joint name="${prefix}palm_tool0" type="fixed">
+        <joint name="${prefix}palm_tool0" type="fixed">
 			<parent link="${prefix}palm"/>
 			<child link="${prefix}tool0"/>
@@ -64,4 +74,25 @@
 		</joint>
 		<!-- end of joint list -->
+__    	<!-- transmission list -->
+        <transmission name="${prefix}palm_finger_1_joint_transmission">
+            <type>transmission_interface/SimpleTransmission</type>
+            <joint name="${prefix}palm_finger_1_joint">
+                <hardwareInterface>hardware_interface/EffortJointInterface</hardwareInterface>
+            </joint>
+            <actuator name="${prefix}palm_finger_1_joint">
+                <hardwareInterface>hardware_interface/EffortJointInterface</hardwareInterface>
+                <mechanicalReduction>1</mechanicalReduction>
+            </actuator>
+        </transmission>
+        <transmission name="${prefix}palm_finger_2_joint_transmission">
+            <type>transmission_interface/SimpleTransmission</type>
+            <joint name="${prefix}palm_finger_2_joint">
+                <hardwareInterface>hardware_interface/EffortJointInterface</hardwareInterface>
+            </joint>
+            <actuator name="${prefix}palm_finger_2_joint">
+                <hardwareInterface>hardware_interface/EffortJointInterface</hardwareInterface>
+                <mechanicalReduction>1</mechanicalReduction>
+            </actuator>
+        </transmission>
 	</xacro:macro>
 </robot>

File: robotiq_3f_gripper_visualization/cfg/robotiq-3f-gripper_finger_articulated_macro.xacro (robot description, xacro)
@@ -1,2 +1,3 @@
+<?xml version="1.0"?>
 <!--
 robotiq-3f-gripper_finder_articulated_macro(prefix)
@@ -32,5 +33,9 @@
                 <inertia ixx="0.01" ixy="-0.00002" ixz="0.00001" iyy="0.0008" iyz="0" izz="0.001" />
             </inertial>
-		</link>
+        </link>
+            <gazebo reference="${prefix}link_0">
+                <mu1>1.1</mu1>
+                <mu2>1.1</mu2>
+            </gazebo>
 		<link name="${prefix}link_1">
 			<visual>
@@ -54,4 +59,8 @@
             </inertial>
 		</link>
+            <gazebo reference="${prefix}link_1">
+                <mu1>1.1</mu1>
+                <mu2>1.1</mu2>
+            </gazebo>
 		<link name="${prefix}link_2">
 			<!--
@@ -80,4 +89,8 @@
             </inertial>
 		</link>
+            <gazebo reference="${prefix}link_2">
+                <mu1>1.1</mu1>
+                <mu2>1.1</mu2>
+            </gazebo>
 		<link name="${prefix}link_3">
 			<visual>
@@ -101,4 +114,8 @@
             </inertial>
 		</link>
+            <gazebo reference="${prefix}link_3">
+                <mu1>1.1</mu1>
+                <mu2>1.1</mu2>
+            </gazebo>
 		<!-- end of link list -->
 		<!-- joint list -->
@@ -125,4 +142,35 @@
 		</joint>
 		<!-- end of joint list -->
-	</xacro:macro>
+    	<!-- transmission list -->
+        <transmission name="${prefix}joint_1_transmission">
+            <type>transmission_interface/SimpleTransmission</type>
+            <joint name="${prefix}joint_1">
+                <hardwareInterface>hardware_interface/EffortJointInterface</hardwareInterface>
+            </joint>
+            <actuator name="${prefix}joint_1">
+                <hardwareInterface>hardware_interface/EffortJointInterface</hardwareInterface>
+                <mechanicalReduction>1</mechanicalReduction>
+            </actuator>
+        </transmission>
+        <transmission name="${prefix}joint_2_transmission">
+            <type>transmission_interface/SimpleTransmission</type>
+            <joint name="${prefix}joint_2">
+                <hardwareInterface>hardware_interface/EffortJointInterface</hardwareInterface>
+            </joint>
+            <actuator name="${prefix}joint_2">
+                <hardwareInterface>hardware_interface/EffortJointInterface</hardwareInterface>
+                <mechanicalReduction>1</mechanicalReduction>
+            </actuator>
+        </transmission>
+        <transmission name="${prefix}joint_3_transmission">
+            <type>transmission_interface/SimpleTransmission</type>
+            <joint name="${prefix}joint_3">
+                <hardwareInterface>hardware_interface/EffortJointInterface</hardwareInterface>
+            </joint>
+            <actuator name="${prefix}joint_3">
+                <hardwareInterface>hardware_interface/EffortJointInterface</hardwareInterface>
+                <mechanicalReduction>1</mechanicalReduction>
+            </actuator>
+        </transmission>
+    </xacro:macro>
 </robot>

Commit message: new interials in acrticulated_marco.xarco and mock intertials in finger macro.xacro. also normal mode in HandPlugin

File: robotiq_3f_gripper_visualization/cfg/robotiq-3f-gripper_actuated_gazebo.xacro (robot description, xacro)
@@ -15,15 +15,15 @@
         <origin xyz="0.057 0.0 0.0" rpy="0.0 ${pi} ${-pi/2}" />
     </joint>
-<!--  <gazebo>
-    <!- - plugin for the RobotiQ hand - ->
-    <plugin name="robotiq_hand_plugin" filename="libRobotiqHandPlugin.so">
-      <kp_position>10.0</kp_position>
-      <kd_position>0.5</kd_position>
-      <!- - Some optional parameters. Check the plugin header file for all of them. - ->
-      <!- -<prefix>pre_</prefix>- ->
-      <!- - This is chosen, so it's compatible with the "Robotiq3FGripperSimpleController.py"- ->
-      <topic_command>/Robotiq3FGripperRobotOutput</topic_command>
-      <!- - <topic_state>/hand/state</topic_state> - ->
-    </plugin>
-  </gazebo> -->
+<!--    <gazebo>
+        <!- - plugin for the RobotiQ hand  - ->
+        <plugin name="robotiq_hand_plugin" filename="libRobotiqHandPlugin.so">
+            <kp_position>10.0</kp_position>
+            <kd_position>0.5</kd_position>
+            <!- - Some optional parameters. Check the plugin header file for all of them. - ->
+            <!- -<prefix>pre_</prefix>- ->
+            <!- - This is chosen, so it's compatible with the "Robotiq3FGripperSimpleController.py"- ->
+            <topic_command>/Robotiq3FGripperRobotOutput</topic_command>
+            <!- - <topic_state>/hand/state</topic_state> - ->
+        </plugin>
+    </gazebo> -->
 </robot>

File: robotiq_3f_gripper_visualization/cfg/robotiq-3f-gripper_articulated_macro.xacro (robot description, xacro)
@@ -30,8 +30,8 @@
 				</material>
 			</collision>
-             <inertial>
-            <origin xyz="0 0 0" rpy="0 0 0"/>
-            <mass value="1.3"/>
-            <inertia ixx="0.0035" ixy="0" ixz="-0" iyy="0.0035" iyz="0" izz="0.0035" />
+            <inertial>
+                <origin xyz="-0.0176262975 -0.0041752643 0.0000287824"/>
+                <mass value="1.3000000000"/>
+                <inertia ixx="0.0022857562" ixy="-0.0000228139" ixz="-0.0000000072" iyy="0.0028530547" iyz="0.0000000027" izz="0.0023702761"/>
             </inertial>
 		</link>
@@ -39,11 +39,14 @@
         <mu1>1.1</mu1>
         <mu2>1.1</mu2>
+        <material>Gazebo/Red</material>
+        <selfCollide>false</selfCollide>
         </gazebo>
-		<link name="${prefix}tool0"/>
-        <inertial>
-            <origin xyz="0 0 0" rpy="0 0 0"/>
-            <mass value="1.3"/>
-            <inertia ixx="0.006012" ixy="0.000079" ixz="-0.00024" iyy="0.012892" iyz="0" izz="0.002435" />
-        </inertial>
+		<link name="${prefix}tool0">
+            <inertial>
+                <origin xyz="-0.0176262975 -0.0041752643 0.0000287824"/>
+                <mass value="0.0010000000"/>
+                <inertia ixx="0.0000017583" ixy="-0.0000000175" ixz="-0.0000000000" iyy="0.0000021947" iyz="0.0000000000" izz="0.0000018233"/>
+            </inertial>
+        </link>
 		<!-- end of link list -->
 		<!-- joint list -->

File: robotiq_3f_gripper_visualization/cfg/robotiq-3f-gripper_finger_articulated_macro.xacro (robot description, xacro)
@@ -31,5 +31,5 @@
                 <origin xyz="0 0 0" rpy="0 0 0"/>
                 <mass value="0.05"/>
-                <inertia ixx="0.01" ixy="-0.00002" ixz="0.00001" iyy="0.0008" iyz="0" izz="0.001" />
+                <inertia ixx="1" ixy="0" ixz="0" iyy="1" iyz="0" izz="1"/>
             </inertial>
         </link>
@@ -37,4 +37,6 @@
                 <mu1>1.1</mu1>
                 <mu2>1.1</mu2>
+                <material>Gazebo/Yellow</material>
+                <selfCollide>false</selfCollide>
             </gazebo>
 		<link name="${prefix}link_1">
@@ -56,5 +58,5 @@
                 <origin xyz="0 0 0" rpy="0 0 0"/>
                 <mass value="0.15"/>
-                <inertia ixx="0.001859" ixy="-0.000376" ixz="0.000028" iyy="0.012756" iyz="0" izz="0.0024" />
+                <inertia ixx="1" ixy="0" ixz="0" iyy="1" iyz="0" izz="1"/>
             </inertial>
 		</link>
@@ -62,4 +64,6 @@
                 <mu1>1.1</mu1>
                 <mu2>1.1</mu2>
+                <material>Gazebo/Green</material>
+                <selfCollide>false</selfCollide>
             </gazebo>
 		<link name="${prefix}link_2">
@@ -86,5 +90,5 @@
                 <origin xyz="0 0 0" rpy="0 0 0"/>
                 <mass value="0.15"/>
-                <inertia ixx="0.001859" ixy="-0.000376" ixz="0.000028" iyy="0.012756" iyz="0" izz="0.0024" />
+                <inertia ixx="1" ixy="0" ixz="0" iyy="1" iyz="0" izz="1"/>
             </inertial>
 		</link>
@@ -92,4 +96,6 @@
                 <mu1>1.1</mu1>
                 <mu2>1.1</mu2>
+                <material>Gazebo/Blue</material>
+                <selfCollide>false</selfCollide>
             </gazebo>
 		<link name="${prefix}link_3">
@@ -111,5 +117,5 @@
                 <origin xyz="0 0 0" rpy="0 0 0"/>
                 <mass value="0.05"/>
-                <inertia ixx="0.001239" ixy="-0.000251" ixz="0.000019" iyy="0.00085" iyz="0" izz="0.001632" />
+                <inertia ixx="1" ixy="0" ixz="0" iyy="1" iyz="0" izz="1"/>
             </inertial>
 		</link>
@@ -117,4 +123,6 @@
                 <mu1>1.1</mu1>
                 <mu2>1.1</mu2>
+                <material>Gazebo/Yellow</material>
+                <selfCollide>false</selfCollide>
             </gazebo>
 		<!-- end of link list -->
@@ -173,4 +181,5 @@
             </actuator>
         </transmission>
-    </xacro:macro>
+	    <!-- end of transmission list -->
+	</xacro:macro>
 </robot>
