Commit message: sensors for fingers in extra xacro file

File: robotiq_3f_gripper_visualization/cfg/robotiq-3f-gripper_articulated.xacro (robot description, xacro)
@@ -7,4 +7,6 @@
         <xacro:include filename="$(find robotiq_3f_gripper_visualization)/cfg/robotiq-3f-gripper_articulated_macro.xacro" />
         <xacro:robotiq-3f-gripper_articulated prefix=""/>
+       <!-- <xacro:include filename="$(find robotiq_3f_gripper_visualization)/cfg/robotiq-3f-gripper_contact-sensors_macro.xacro" />
+        <xacro:robotiq-3f-gripper_articulated prefix=""/> -->
 <!--
         <xacro:include filename="$(find robotiq_3f_gripper_visualization)/cfg/robotiq-3f-gripper_finger_articulated_macro.xacro" />

File: robotiq_3f_gripper_visualization/cfg/robotiq-3f-gripper_articulated_macro.xacro (robot description, xacro)
@@ -1,3 +1,3 @@
-<?xml version="1.0"?>
+<?xml version="1.0" ?>
 <!--
 robotiq-3f-gripper_articulated_macro(prefix)
@@ -8,4 +8,6 @@
 <robot xmlns:xacro="http://ros.org/wiki/xacro">
         <xacro:include filename="$(find robotiq_3f_gripper_visualization)/cfg/robotiq-3f-gripper_finger_articulated_macro.xacro" />
+		<xacro:include filename="$(find robotiq_3f_gripper_visualization)/cfg/robotiq-3f-gripper_contact-sensors_macro.xacro" />
+		<xacro:robotiq-3f-gripper_contact-sensors prefix=""/>
         <xacro:macro name="robotiq-3f-gripper_articulated" params="prefix">
         <xacro:robotiq-3f-gripper_finger_articulated prefix="${prefix}finger_1_"/>
@@ -24,5 +26,5 @@
 			<collision>
 				<geometry>
-                                        <mesh filename="package://robotiq_3f_gripper_visualization/meshes/robotiq-3f-gripper_articulated/collision/palm.STL" />
+                                        <mesh filename="package://robotiq_3f_gripper_visualization/meshes/robotiq-3f-gripper_articulated/collision/palm_with_finger_cutouts.stl" />
 				</geometry>
 				<material name="yellow">
@@ -30,23 +32,11 @@
 				</material>
 			</collision>
-            <inertial>
-                <origin xyz="-0.0176262975 -0.0041752643 0.0000287824"/>
-                <mass value="1.3000000000"/>
-                <inertia ixx="0.0022857562" ixy="-0.0000228139" ixz="-0.0000000072" iyy="0.0028530547" iyz="0.0000000027" izz="0.0023702761"/>
-            </inertial>
 		</link>
-        <gazebo reference="${prefix}palm">
-        <mu1>1.1</mu1>
-        <mu2>1.1</mu2>
-        <material>Gazebo/Red</material>
-        <selfCollide>false</selfCollide>
-        </gazebo>
-		<link name="${prefix}tool0">
-            <inertial>
-                <origin xyz="-0.0176262975 -0.0041752643 0.0000287824"/>
-                <mass value="0.0010000000"/>
-                <inertia ixx="0.0000017583" ixy="-0.0000000175" ixz="-0.0000000000" iyy="0.0000021947" iyz="0.0000000000" izz="0.0000018233"/>
-            </inertial>
-        </link>
+		<link name="${prefix}tool0"/>
+        <inertial>
+            <origin xyz="0 0 0" rpy="0 0 0"/>
+            <mass value="1.3"/>
+            <inertia ixx="0.006012" ixy="0.000079" ixz="-0.00024" iyy="0.012892" iyz="0" izz="0.002435" />
+        </inertial>
 		<!-- end of link list -->
 		<!-- joint list -->
@@ -56,5 +46,6 @@
 			<axis xyz="0 1 0"/>
 			<origin xyz="-0.0455 0.0214 0.036" rpy="0 3.1416 -1.57"/>
-			<limit lower="-0.1784" upper="0.192" effort="100" velocity="100"/>
+			<limit lower="-0.1784" upper="0.192" effort="100" velocity="1.23"/>
+      <dynamics friction="0.1" damping="1.0" />
 		</joint>
 		<joint name="${prefix}palm_finger_2_joint" type="revolute">
@@ -63,5 +54,6 @@
 			<axis xyz="0 1 0"/>
 			<origin xyz="-0.0455 0.0214 -0.036" rpy="0 3.1416 -1.57"/>
-			<limit lower="-0.192" upper="0.1784" effort="100" velocity="100"/>
+			<limit lower="-0.192" upper="0.1784" effort="100" velocity="1.23"/>
+      <dynamics friction="0.1" damping="1.0" />
 		</joint>
 		<joint name="${prefix}palm_finger_middle_joint" type="fixed">
@@ -71,5 +63,5 @@
 			<origin xyz="0.0455 0.0214 0" rpy="0 0 1.57"/>
 		</joint>
-        <joint name="${prefix}palm_tool0" type="fixed">
+		<joint name="${prefix}palm_tool0" type="fixed">
 			<parent link="${prefix}palm"/>
 			<child link="${prefix}tool0"/>
@@ -77,25 +69,4 @@
 		</joint>
 		<!-- end of joint list -->
-__    	<!-- transmission list -->
-        <transmission name="${prefix}palm_finger_1_joint_transmission">
-            <type>transmission_interface/SimpleTransmission</type>
-            <joint name="${prefix}palm_finger_1_joint">
-                <hardwareInterface>hardware_interface/EffortJointInterface</hardwareInterface>
-            </joint>
-            <actuator name="${prefix}palm_finger_1_joint">
-                <hardwareInterface>hardware_interface/EffortJointInterface</hardwareInterface>
-                <mechanicalReduction>1</mechanicalReduction>
-            </actuator>
-        </transmission>
-        <transmission name="${prefix}palm_finger_2_joint_transmission">
-            <type>transmission_interface/SimpleTransmission</type>
-            <joint name="${prefix}palm_finger_2_joint">
-                <hardwareInterface>hardware_interface/EffortJointInterface</hardwareInterface>
-            </joint>
-            <actuator name="${prefix}palm_finger_2_joint">
-                <hardwareInterface>hardware_interface/EffortJointInterface</hardwareInterface>
-                <mechanicalReduction>1</mechanicalReduction>
-            </actuator>
-        </transmission>
 	</xacro:macro>
 </robot>

File: robotiq_3f_gripper_visualization/cfg/robotiq-3f-gripper_finger_articulated_macro.xacro (robot description, xacro)
@@ -1,3 +1,3 @@
-<?xml version="1.0"?>
+<?xml version="1.0" ?>
 <!--
 robotiq-3f-gripper_finder_articulated_macro(prefix)
@@ -31,13 +31,7 @@
                 <origin xyz="0 0 0" rpy="0 0 0"/>
                 <mass value="0.05"/>
-                <inertia ixx="1" ixy="0" ixz="0" iyy="1" iyz="0" izz="1"/>
+                <inertia ixx="0.01" ixy="-0.00002" ixz="0.00001" iyy="0.0008" iyz="0" izz="0.001" />
             </inertial>
-        </link>
-            <gazebo reference="${prefix}link_0">
-                <mu1>1.1</mu1>
-                <mu2>1.1</mu2>
-                <material>Gazebo/Yellow</material>
-                <selfCollide>false</selfCollide>
-            </gazebo>
+            </link>
 		<link name="${prefix}link_1">
 			<visual>
@@ -48,5 +42,5 @@
 				<material name="gray"/>
 			</visual>
-			<collision>
+			<collision name="collision_link_1">
 				<origin xyz="0.050 -.028 0" rpy="0 0 -0.52"/>
 				<geometry>
@@ -58,13 +52,7 @@
                 <origin xyz="0 0 0" rpy="0 0 0"/>
                 <mass value="0.15"/>
-                <inertia ixx="1" ixy="0" ixz="0" iyy="1" iyz="0" izz="1"/>
+                <inertia ixx="0.001859" ixy="-0.000376" ixz="0.000028" iyy="0.012756" iyz="0" izz="0.0024" />
             </inertial>
-		</link>
-            <gazebo reference="${prefix}link_1">
-                <mu1>1.1</mu1>
-                <mu2>1.1</mu2>
-                <material>Gazebo/Green</material>
-                <selfCollide>false</selfCollide>
-            </gazebo>
+        </link>
 		<link name="${prefix}link_2">
 			<!--
@@ -90,13 +78,7 @@
                 <origin xyz="0 0 0" rpy="0 0 0"/>
                 <mass value="0.15"/>
-                <inertia ixx="1" ixy="0" ixz="0" iyy="1" iyz="0" izz="1"/>
+                <inertia ixx="0.001859" ixy="-0.000376" ixz="0.000028" iyy="0.012756" iyz="0" izz="0.0024" />
             </inertial>
 		</link>
-            <gazebo reference="${prefix}link_2">
-                <mu1>1.1</mu1>
-                <mu2>1.1</mu2>
-                <material>Gazebo/Blue</material>
-                <selfCollide>false</selfCollide>
-            </gazebo>
 		<link name="${prefix}link_3">
 			<visual>
@@ -117,14 +99,7 @@
                 <origin xyz="0 0 0" rpy="0 0 0"/>
                 <mass value="0.05"/>
-                <inertia ixx="1" ixy="0" ixz="0" iyy="1" iyz="0" izz="1"/>
+                <inertia ixx="0.001239" ixy="-0.000251" ixz="0.000019" iyy="0.00085" iyz="0" izz="0.001632" />
             </inertial>
 		</link>
-            <gazebo reference="${prefix}link_3">
-                <mu1>1.1</mu1>
-                <mu2>1.1</mu2>
-                <material>Gazebo/Yellow</material>
-                <selfCollide>false</selfCollide>
-            </gazebo>
-		<!-- end of link list -->
 		<!-- joint list -->
 		<joint name="${prefix}joint_1" type="revolute">
@@ -133,5 +108,7 @@
 			<axis xyz="0 0 1"/>
 			<origin xyz="0.020 0 0" rpy="0 0 0"/>
-			<limit lower="0.0495" upper="1.2218" effort="100" velocity="100"/>
+      <!-- fnh: velocity=100 is far too fast. We also want some damping for Gazebo -->
+			<limit lower="0.0495" upper="1.2218" effort="100" velocity="1.23"/>
+      <dynamics friction="0.1" damping="1"/>
 		</joint>
 		<joint name="${prefix}joint_2" type="revolute">
@@ -140,5 +117,6 @@
 			<axis xyz="0 0 1"/>
 			<origin xyz="0.050 -.028 0" rpy="0 0 -0.52"/>
-			<limit lower="0.0" upper="1.5708" effort="100" velocity="100"/>
+			<limit lower="0.0" upper="1.5708" effort="100" velocity="1.24"/>
+      <dynamics friction="0.1" damping="1"/>
 		</joint>
 		<joint name="${prefix}joint_3" type="revolute">
@@ -147,39 +125,8 @@
 			<axis xyz="0 0 1"/>
 			<origin xyz="0.039 0 0" rpy="0 0 0"/>
-			<limit lower="-1.2217" upper="-0.0523" effort="100" velocity="100"/>
+			<limit lower="-1.2217" upper="-0.0523" effort="100" velocity="1.25"/>
+      <dynamics friction="0.1" damping="1"/>
 		</joint>
 		<!-- end of joint list -->
-    	<!-- transmission list -->
-        <transmission name="${prefix}joint_1_transmission">
-            <type>transmission_interface/SimpleTransmission</type>
-            <joint name="${prefix}joint_1">
-                <hardwareInterface>hardware_interface/EffortJointInterface</hardwareInterface>
-            </joint>
-            <actuator name="${prefix}joint_1">
-                <hardwareInterface>hardware_interface/EffortJointInterface</hardwareInterface>
-                <mechanicalReduction>1</mechanicalReduction>
-            </actuator>
-        </transmission>
-        <transmission name="${prefix}joint_2_transmission">
-            <type>transmission_interface/SimpleTransmission</type>
-            <joint name="${prefix}joint_2">
-                <hardwareInterface>hardware_interface/EffortJointInterface</hardwareInterface>
-            </joint>
-            <actuator name="${prefix}joint_2">
-                <hardwareInterface>hardware_interface/EffortJointInterface</hardwareInterface>
-                <mechanicalReduction>1</mechanicalReduction>
-            </actuator>
-        </transmission>
-        <transmission name="${prefix}joint_3_transmission">
-            <type>transmission_interface/SimpleTransmission</type>
-            <joint name="${prefix}joint_3">
-                <hardwareInterface>hardware_interface/EffortJointInterface</hardwareInterface>
-            </joint>
-            <actuator name="${prefix}joint_3">
-                <hardwareInterface>hardware_interface/EffortJointInterface</hardwareInterface>
-                <mechanicalReduction>1</mechanicalReduction>
-            </actuator>
-        </transmission>
-	    <!-- end of transmission list -->
 	</xacro:macro>
 </robot>

File: robotiq_3f_gripper_visualization/cfg/robotiq-3f-gripper_mesh_macro.xacro (robot description, xacro)
@@ -1,2 +1,3 @@
+<?xml version="1.0" ?>
 <robot xmlns:xacro="http://ros.org/wiki/xacro">
         <xacro:macro name="robotiq-3f-gripper_mesh" params="prefix">
