Commit message: last minor changes

File: robotiq_3f_gripper_visualization/cfg/robotiq-3f-gripper_contact-sensors_macro.xacro (robot description, xacro)
@@ -12,5 +12,5 @@
                 <origin xyz="0 0 0" rpy="0 0 0" />
                 <geometry>
-                    <box size="0.03 0.0001 0.02" />
+                    <box size="0.04 0.001 0.03" /> <!--0.027-->
                 </geometry>
             </visual>
@@ -18,5 +18,5 @@
                 <origin xyz="0 0 0" rpy="0 0 0" />
                 <geometry>
-                    <box size="0.01 0.01 0.02" />
+                    <box size="0.04 0.001 0.03" />
                 </geometry>
             </collision>
@@ -47,5 +47,5 @@
                 <origin xyz="0 0 0" rpy="0 0 0" />
                 <geometry>
-                    <box size="0.02 0.0001 0.02" />
+                    <box size="0.033 0.001 0.03" />
                 </geometry>
             </visual>
@@ -53,5 +53,5 @@
                 <origin xyz="0 0 0" rpy="0 0 0" />
                 <geometry>
-                    <box size="0.02 0.0001 0.02" />
+                    <box size="0.033 0.001 0.03" />
                 </geometry>
             </collision>
@@ -82,5 +82,5 @@
                 <origin xyz="0 0 0" rpy="0 0 0" />
                 <geometry>
-                    <box size="0.02 0.0001 0.02" />
+                    <box size="0.02 0.001 0.025" />
                 </geometry>
             </visual>
@@ -88,5 +88,5 @@
                 <origin xyz="0 0 0" rpy="0 0 0" />
                 <geometry>
-                    <box size="0.02 0.0001 0.02" />
+                    <box size="0.02 0.001 0.025" />
                 </geometry>
             </collision>
@@ -117,5 +117,5 @@
                 <origin xyz="0 0 0" rpy="0 0 0" />
                 <geometry>
-                    <box size="0.03 0.0001 0.02" />
+                    <box size="0.04 0.001 0.03" />
                 </geometry>
             </visual>
@@ -123,5 +123,5 @@
                 <origin xyz="0 0 0" rpy="0 0 0" />
                 <geometry>
-                    <box size="0.01 0.01 0.02" />
+                    <box size="0.04 0.001 0.03" />
                 </geometry>
             </collision>
@@ -152,5 +152,5 @@
                 <origin xyz="0 0 0" rpy="0 0 0" />
                 <geometry>
-                    <box size="0.03 0.0001 0.02" />
+                    <box size="0.033 0.001 0.03" />
                 </geometry>
             </visual>
@@ -158,5 +158,5 @@
                 <origin xyz="0 0 0" rpy="0 0 0" />
                 <geometry>
-                    <box size="0.01 0.01 0.02" />
+                    <box size="0.033 0.001 0.03" />
                 </geometry>
             </collision>
@@ -187,5 +187,5 @@
                 <origin xyz="0 0 0" rpy="0 0 0" />
                 <geometry>
-                    <box size="0.02 0.0001 0.02" />
+                    <box size="0.02 0.001 0.025" />
                 </geometry>
             </visual>
@@ -193,5 +193,5 @@
                 <origin xyz="0 0 0" rpy="0 0 0" />
                 <geometry>
-                    <box size="0.02 0.0001 0.02" />
+                    <box size="0.02 0.001 0.025" />
                 </geometry>
             </collision>
@@ -222,5 +222,5 @@
                 <origin xyz="0 0 0" rpy="0 0 0" />
                 <geometry>
-                    <box size="0.03 0.0001 0.02" />
+                    <box size="0.04 0.001 0.03" />
                 </geometry>
             </visual>
@@ -228,5 +228,5 @@
                 <origin xyz="0 0 0" rpy="0 0 0" />
                 <geometry>
-                    <box size="0.01 0.01 0.02" />
+                    <box size="0.04 0.001 0.03" />
                 </geometry>
             </collision>
@@ -257,5 +257,5 @@
                 <origin xyz="0 0 0" rpy="0 0 0" />
                 <geometry>
-                    <box size="0.03 0.0001 0.02" />
+                    <box size="0.033 0.001 0.03" />
                 </geometry>
             </visual>
@@ -263,5 +263,5 @@
                 <origin xyz="0 0 0" rpy="0 0 0" />
                 <geometry>
-                    <box size="0.01 0.01 0.02" />
+                    <box size="0.033 0.001 0.03" />
                 </geometry>
             </collision>
@@ -292,5 +292,5 @@
                 <origin xyz="0 0 0" rpy="0 0 0" />
                 <geometry>
-                    <box size="0.02 0.0001 0.02" />
+                    <box size="0.02 0.001 0.025" />
                 </geometry>
             </visual>
@@ -298,5 +298,5 @@
                 <origin xyz="0 0 0" rpy="0 0 0" />
                 <geometry>
-                    <box size="0.02 0.0001 0.02" />
+                    <box size="0.02 0.001 0.025" />
                 </geometry>
             </collision>
@@ -328,5 +328,5 @@
             <child link="s_model_finger_1_link_1_sensor"/>
             <!-- <origin xyz="0.020 0 0" rpy="0 0 0"/> -->
-			<origin xyz="0.04 -0.0127 0" rpy="0 0 -0.61"/>
+			<origin xyz="0.04 -0.014 0" rpy="0 0 -0.52"/>
         </joint>
 		<joint name="s_model_finger_1_link_2_sensor_joint" type="fixed">
@@ -334,5 +334,5 @@
             <child link="s_model_finger_1_link_2_sensor"/>
             <!-- <origin xyz="0.020 0 0" rpy="0 0 0"/> -->
-			<origin xyz="0.02 0.008 0" rpy="0 0 0.015"/>
+			<origin xyz="0.022 0.0075 0" rpy="0 0 0.0"/>
         </joint>
 		<joint name="s_model_finger_1_link_3_sensor_joint" type="fixed">
@@ -341,35 +341,35 @@
             <!-- <origin xyz="0.020 0 0" rpy="0 0 0"/> -->
 			<!-- <origin xyz="0.04 -0.0127 0" rpy="0 0 -0.61"/> -->
-			<origin xyz="0.018 0.0198 0" rpy="0 0 0.51"/>
+			<origin xyz="0.0181 0.0196 0" rpy="0 0 0.505"/>
         </joint>
 		<joint name="s_model_finger_2_link_1_sensor_joint" type="fixed">
             <parent link="s_model_finger_2_link_1"/>
             <child link="s_model_finger_2_link_1_sensor"/>
-			<origin xyz="0.04 -0.0127 0" rpy="0 0 -0.61"/>
+			<origin xyz="0.04 -0.014 0" rpy="0 0 -0.52"/>
         </joint>
 		<joint name="s_model_finger_2_link_2_sensor_joint" type="fixed">
             <parent link="s_model_finger_2_link_2"/>
             <child link="s_model_finger_2_link_2_sensor"/>
-			<origin xyz="0.02 0.008 0" rpy="0 0 0.015"/>
+			<origin xyz="0.022 0.0075 0" rpy="0 0 0.0"/>
         </joint>
 		<joint name="s_model_finger_2_link_3_sensor_joint" type="fixed">
             <parent link="s_model_finger_2_link_3"/>
             <child link="s_model_finger_2_link_3_sensor"/>
-			<origin xyz="0.018 0.0198 0" rpy="0 0 0.51"/>
+			<origin xyz="0.0181 0.0196 0" rpy="0 0 0.505"/>
         </joint>
 		<joint name="s_model_finger_middle_link_1_sensor_joint" type="fixed">
             <parent link="s_model_finger_middle_link_1"/>
             <child link="s_model_finger_middle_link_1_sensor"/>
-			<origin xyz="0.04 -0.0127 0" rpy="0 0 -0.61"/>
+			<origin xyz="0.04 -0.014 0" rpy="0 0 -0.52"/>
         </joint>
 		<joint name="s_model_finger_middle_link_2_sensor_joint" type="fixed">
             <parent link="s_model_finger_middle_link_2"/>
             <child link="s_model_finger_middle_link_2_sensor"/>
-			<origin xyz="0.02 0.008 0" rpy="0 0 0.015"/>
+			<origin xyz="0.022 0.0075 0" rpy="0 0 0.0"/>
         </joint>
 		<joint name="s_model_finger_middle_link_3_sensor_joint" type="fixed">
             <parent link="s_model_finger_middle_link_3"/>
             <child link="s_model_finger_middle_link_3_sensor"/>
-			<origin xyz="0.018 0.0198 0" rpy="0 0 0.51"/>
+			<origin xyz="0.0181 0.0196 0" rpy="0 0 0.505"/>
         </joint>
         <!-- end of sensor joint list-->

File: robotiq_3f_gripper_visualization/cfg/robotiq-3f-gripper_finger_articulated_macro.xacro (robot description, xacro)
@@ -45,5 +45,6 @@
 				<origin xyz="0.050 -.028 0" rpy="0 0 -0.52"/>
 				<geometry>
-                                        <mesh filename="package://robotiq_3f_gripper_visualization/meshes/robotiq-3f-gripper_articulated/collision/link_1.STL" />
+                                        <!-- <mesh filename="package://robotiq_3f_gripper_visualization/meshes/robotiq-3f-gripper_articulated/collision/link_1.STL" /> -->
+										<mesh filename="package://robotiq_3f_gripper_visualization/meshes/robotiq-3f-gripper_articulated/visual/link_1.dae" />
 				</geometry>
 				<material name="yellow"/>
@@ -71,5 +72,6 @@
 				<origin xyz="0.039 0 0.0075" rpy="0 0 0"/>
 				<geometry>
-                                        <mesh filename="package://robotiq_3f_gripper_visualization/meshes/robotiq-3f-gripper_articulated/collision/link_2.STL" />
+                                        <!-- <mesh filename="package://robotiq_3f_gripper_visualization/meshes/robotiq-3f-gripper_articulated/collision/link_2.STL" /> -->
+										<mesh filename="package://robotiq_3f_gripper_visualization/meshes/robotiq-3f-gripper_articulated/visual/link_2.dae" />
 				</geometry>
 				<material name="yellow"/>
@@ -92,5 +94,6 @@
 				<origin xyz="0 0 0" rpy="0 0 0.52"/>
 				<geometry>
-                                        <mesh filename="package://robotiq_3f_gripper_visualization/meshes/robotiq-3f-gripper_articulated/collision/link_3.STL" />
+                                      <!--  <mesh filename="package://robotiq_3f_gripper_visualization/meshes/robotiq-3f-gripper_articulated/collision/link_3.STL" /> -->
+									  <mesh filename="package://robotiq_3f_gripper_visualization/meshes/robotiq-3f-gripper_articulated/visual/link_3.dae" />
 				</geometry>
 				<material name="yellow"/>
@@ -109,5 +112,5 @@
 			<origin xyz="0.020 0 0" rpy="0 0 0"/>
       <!-- fnh: velocity=100 is far too fast. We also want some damping for Gazebo -->
-			<limit lower="0.0495" upper="1.2218" effort="100" velocity="1.23"/>
+			<limit lower="0.0495" upper="1.2218" effort="90" velocity="1.23"/>
       <dynamics friction="0.1" damping="1"/>
 		</joint>
@@ -117,5 +120,5 @@
 			<axis xyz="0 0 1"/>
 			<origin xyz="0.050 -.028 0" rpy="0 0 -0.52"/>
-			<limit lower="0.0" upper="1.5708" effort="100" velocity="1.24"/>
+			<limit lower="0.0" upper="1.5708" effort="90" velocity="1.24"/>
       <dynamics friction="0.1" damping="1"/>
 		</joint>
@@ -125,5 +128,5 @@
 			<axis xyz="0 0 1"/>
 			<origin xyz="0.039 0 0" rpy="0 0 0"/>
-			<limit lower="-1.2217" upper="-0.0523" effort="100" velocity="1.25"/>
+			<limit lower="-1.2217" upper="-0.0523" effort="90" velocity="1.25"/>
       <dynamics friction="0.1" damping="1"/>
 		</joint>
